Commit message: wip - spot mdp

File: workspace/gym_ignition_description/gym_ignition_models/spot/spot.urdf (robot description, URDF)
Before this commit: robot spot, 20 links, 19 joints
Links:
- link body: geometry collision box size=0.86 0.21 0.17; visual mesh filename=model://spot/meshes/visual/body.dae
- link front_left_hip: geometry visual mesh filename=model://spot/meshes/visual/front_left_hip.dae
- link front_left_lower_leg: geometry collision cylinder length=0.252 radius=0.035; visual mesh filename=model://spot/meshes/visual/front_left_lower_leg.dae
- link front_left_upper_leg: geometry collision cylinder length=0.34 radius=0.0456; visual mesh filename=model://spot/meshes/visual/front_left_upper_leg.dae
- link front_right_hip: geometry visual mesh filename=model://spot/meshes/visual/front_right_hip.dae
- link front_right_lower_leg: geometry collision cylinder length=0.252 radius=0.035; visual mesh filename=model://spot/meshes/visual/front_right_lower_leg.dae
- link front_right_upper_leg: geometry collision cylinder length=0.34 radius=0.0456; visual mesh filename=model://spot/meshes/visual/front_right_upper_leg.dae
- link rear_left_hip: geometry visual mesh filename=model://spot/meshes/visual/rear_left_hip.dae
- link rear_left_lower_leg: geometry collision cylinder length=0.252 radius=0.035; visual mesh filename=model://spot/meshes/visual/rear_left_lower_leg.dae
- link rear_left_upper_leg: geometry collision cylinder length=0.34 radius=0.0456; visual mesh filename=model://spot/meshes/visual/rear_left_upper_leg.dae
- link rear_right_hip: geometry visual mesh filename=model://spot/meshes/visual/rear_right_hip.dae
- link rear_right_lower_leg: geometry collision cylinder length=0.252 radius=0.035; visual mesh filename=model://spot/meshes/visual/rear_right_lower_leg.dae
- link rear_right_upper_leg: geometry collision cylinder length=0.34 radius=0.0456; visual mesh filename=model://spot/meshes/visual/rear_right_upper_leg.dae
